File: KiCAD_Project/Digital_PCB.kicad_pcb (KiCad board)
At the start: 4 copper layers, 75 x 84.8 mm, 112 parts, among them J1 NP_Conn_01x02_Relief, J10 NP_Conn_01x02_Relief, J11 1-0000050, J12 1-0000190, J2 Board to Board, J3 1-0001156, J4 1-0001205, J5 1-0001156, J6 NP_Conn_01x04, J7 NP_Conn_01x02_Relief, J8 NP_Conn_01x04, J9 NP_Conn_01x02_Relief, Q1 1-0001670, U1 1-0000207, U10 1-0000785, U11 1-0000464, U2 1-0000465, U3 1-0000576, U4 1-0001530, U5 1-0001542, U6 1-0001471, U7 1-0000264, U8 1-0000264, U9 1-0001535, Y1 1-0000721

Commit message: Rev 2.1 Changes: - Fixed Issue #11 (U4 Footprint pin 1 indicator) - Added Open Log Header for breakout - Removed SD Circuit - Connected GPS to I2C - Updated IPN and Revision Number
Parts:
- removed C29: 1-0000007, capacitors_0603:1-0000007
- removed the J12 at (175.1, 77.3)
- removed the R12 at (165.2, 88.1)
- removed the R38 at (166.0, 72.0)
- removed the R39 at (166.0, 81.3)
- removed the R9 at (165.2, 86.6)
- added J6: NP_Conn_01x06, np_connectors:PinHeader_1x06_P2.54mm_Vertical, F.Cu at (164.1, 68.5)
- added R1: 1-0000006, resistors_0603:1-0000006, F.Cu at (161.9, 87.1)
- added R2: 1-0000006, resistors_0603:1-0000006, F.Cu at (160.4, 87.1)
- added R3: 1-0000006, resistors_0603:1-0000006, F.Cu at (158.9, 87.1)
- added R4: 1-0000006, resistors_0603:1-0000006, F.Cu at (157.4, 87.1)
- moved R7 9.61 mm to (136.9, 82.3), turned to 0 degrees
- moved R6 7.54 mm to (136.9, 83.9), turned to 0 degrees
- moved C14 5.53 mm to (136.9, 85.4), turned to 0 degrees
- moved C10 4.95 mm to (152.4, 93.2)
- moved C15 4.95 mm to (148.5, 76.8)
- moved C16 4.95 mm to (155.6, 76.8)
- moved C17 4.95 mm to (139.8, 76.8)
- moved C18 4.95 mm to (146.9, 76.8)
- moved C20 4.95 mm to (156.5, 72.1)
- moved C21 4.95 mm to (156.5, 73.7)
- moved C9 4.95 mm to (152.4, 88.9)
- moved R25 4.95 mm to (142.4, 85.0)
- moved R26 4.95 mm to (145.4, 85.0)
- moved R27 4.95 mm to (143.9, 85.0)
- moved R28 4.95 mm to (148.5, 85.0)
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- renumbered C27 to C26, C26 to C27, J9 to J10, J10 to J11, J11 to J12, J6 to J7, J7 to J8, J8 to J9, R11 to R10, R5 to R11, R6 to R12, R7 to R15, R8 to R19, R15 to R20, R19 to R21, R20 to R22, R21 to R23, R22 to R24, R23 to R25, R24 to R26, R25 to R27, R26 to R28, R27 to R29, R28 to R30, R29 to R31, R30 to R32, R31 to R33, R32 to R34, R33 to R35, R35 to R36, R36 to R37, R34 to R38, R37 to R39, R1 to R5, R2 to R6, R3 to R7, R4 to R8, R10 to R9
Connections:
- U1 pad 40: SD_CD -> unconnected-(U1-PB4-Pad40)
- U1 pad 41: SD_CS -> unconnected-(U1-PB5-Pad41)
- U11 pad 16: unconnected-(U11-SDA-Pad16) -> I2C_SDA
- U11 pad 17: unconnected-(U11-SCL-Pad17) -> I2C_SCL
Routing:
- net SD_CD: track 44.7 -> 0.00 mm
- net SD_CS: track 33.6 -> 0.00 mm
- net I2C_SDA: track 97.5 -> 129.0 mm, vias 2 -> 4
- net SPI_MISO: track 51.4 -> 22.2 mm
- net SPI_SCK: track 50.2 -> 22.4 mm, vias 4 -> 2
- net I2C_SCL: track 95.3 -> 123.1 mm, vias 4 -> 5
- net Radio_TX: track 57.7 -> 85.0 mm, vias 1 -> 3
- net SPI_MOSI: track 47.5 -> 22.8 mm
- net Radio_RX: track 61.5 -> 84.4 mm, vias 1 -> 3
- net +3V3: track 86.8 -> 68.9 mm, vias 24 -> 22
- net Net-(J6-Pin_4): track 0.00 -> 15.7 mm
- net Net-(J6-Pin_5): track 0.00 -> 13.4 mm
- net GND: track 123.3 -> 113.8 mm, vias 56 -> 50
- net Yacc: track 109.9 -> 104.9 mm
- net Zacc: track 91.2 -> 86.3 mm
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Other:
- board text added: "3-0000279"
- board text added: "Leeman Geophysical LLC Digital Rotating Electronics Rev 2.1"
- board text added: "Open Log"
- board text removed: "3-0000270"
- board text removed: "Leeman Geophysical LLC Digital Rotating Electronics Rev 2.0"
